File: gamma_carrier/power.kicad_sch (KiCad schematic)
At the start: 8 parts

Commit message: lm5116 done, not checked yet
Parts:
- added Cboot: 100n, symbol Device:C
- added Ccomp: 190p, symbol Device:C
- added Ccomp2: 12p, symbol Device:C
- added Cout: 47u, symbol Device:C
- added Cvcc: 1u, symbol Device:C
- added D1: 1N4148WT, Diode_SMD:D_SOD-523, symbol Diode:1N4148WT
- added L1: 2.8u, symbol Device:L
- added Q1, Q2: NMOS, symbol Simulation_SPICE:NMOS
- added R2: 34.7k, symbol Device:R
- added R3: 11.7k, symbol Device:R
- added Rcomp: 59k, symbol Device:R
- added Rsense: 6m, symbol Device:R
- added Ruv2: 2.49k, symbol Device:R
- renumbered R1 to Ruv1
Connections:
- net GND: now also LM5116.11 (DEMB), LM5116.13 (CSG), LM5116.14 (PGND), Cout.2, Cvcc.2, R3.2, Rsense.2, Ruv2.2
- net VIN: now also Q1.1 (D)
- net at LM5116.10 (VOUT): now also Cout.1, L1.2, R2.1
- net at LM5116.12 (CS): now also Q2.3 (S), Rsense.1
- net at LM5116.15 (LO): now also Q2.2 (G)
- net at LM5116.16 (VCC): now also Cvcc.1, D1.2 (A)
- net at LM5116.18 (HB): now also Cboot.1, D1.1 (K)
- net at LM5116.19 (HO): now also Q1.2 (G)
- net at LM5116.2 (UVLO), Ruv1.1: now also Ruv2.1
- net at LM5116.20 (SW): now also Cboot.2, L1.1, Q1.3 (S), Q2.1 (D)
- net at LM5116.8 (FB): now also Ccomp.2, Ccomp2.1
- net at LM5116.9 (COMP): now also Ccomp2.2, Rcomp.2
- new net: Ccomp.1, Rcomp.1
- new net: R2.2, R3.1
Other:
- moved on the sheet: CSS, C_ramp, Cin, Cin_x, R_EN, R_t, Ruv1

Commit message: attempted to put jetsons onto kicad
Parts:
- LM5116: footprint (none) -> Package_SO:HTSSOP-20-1EP_4.4x6.5mm_P0.65mm_EP3.4x4mm
- renumbered CSS to CSS1, C_ramp to C_ramp1, Cboot to Cboot1, Ccomp to Ccomp1, Cin to Cin1, Cin_x to Cin_x1, Cout to Cout1, Cvcc to Cvcc1, R_EN to R_EN1, R_t to R_t1, Rcomp to Rcomp1, Rsense to Rsense1
Connections:
- net GND: now also LM5116.21 (EP)
- net +5V: now reaches Cout1.1, L1.2, LM5116.10 (VOUT), R2.1

Commit message: jetson power done, need fan and revision
Connections:
- net +5V renamed +5V_JETSON
Changed lines of the file:
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@@
-	)
-	(junction
-		(at 224.79 68.58)
-		(diameter 0)
-		(color 0 0 0 0)
 	)
 	(junction
@@
 	)
 	(junction
+		(at 247.65 68.58)
+		(diameter 0)
+		(color 0 0 0 0)
+	)
+	(junction
 		(at 52.07 57.15)
 		(diameter 0)
@@
 	(wire
 		(pts
-			(xy 224.79 68.58) (xy 218.44 68.58)
+			(xy 218.44 68.58) (xy 232.41 68.58)
 		)
 		(stroke
@@
 	(wire
 		(pts
-			(xy 232.41 68.58) (xy 224.79 68.58)
-		)
-		(stroke
-			(width 0)
-			(type default)
-		)
-	)
-	(wire
-		(pts
 			(xy 161.29 109.22) (xy 176.53 109.22)
 		)
@@
 			(width 0)
 			(type default)
-		)
-	)
-	(label "5VO_SYS"
-		(at 237.49 68.58 0)
-		(effects
-			(font
-				(size 1.27 1.27)
-			)
-			(justify left bottom)
 		)
 	)
@@
 	)
 	(symbol
+		(lib_id "power:PWR_FLAG")
+		(at 232.41 68.58 0)
+		(unit 1)
+		(exclude_from_sim no)
+		(in_bom yes)
+		(on_board yes)
+		(dnp no)
+		(fields_autoplaced yes)
+		(property "Reference" "#FLG02"
+			(at 232.41 66.675 0)
+			(effects
+				(font
+					(size 1.27 1.27)
+				)
+				(hide yes)
+			)
+		)
+		(property "Value" "PWR_FLAG"
+			(at 232.41 63.5 0)
+			(effects
+				(font
+					(size 1.27 1.27)
+				)
+			)
+		)
+		(property "Footprint" ""
+			(at 232.41 68.58 0)
+			(effects
+				(font
+					(size 1.27 1.27)
+				)
+				(hide yes)
+			)
+		)
+		(property "Datasheet" "~"
+			(at 232.41 68.58 0)
+			(effects
+				(font
+					(size 1.27 1.27)
+				)
+				(hide yes)
+			)
+		)
+		(property "Description" "Special symbol for telling ERC where power comes from"
+			(at 232.41 68.58 0)
+			(effects
+				(font
+					(size 1.27 1.27)
+				)
+				(hide yes)
+			)
+		)
+		(pin "1"
+		)
+		(instances
+			(project ""
+				(path "/14709545-fb6c-4e0b-b295-f7f5e8a286ba/0e58818c-005b-4d62-adc6-0567728bdecf"
+					(reference "#FLG02")
+					(unit 1)
+				)
+			)
+		)
+	)
+	(symbol
 		(lib_id "power:GND")
 		(at 91.44 100.33 0)
@@
 	)
 	(symbol
+		(lib_id "gamma_lib:+5V_JETSON")
+		(at 247.65 68.58 0)
+		(unit 1)
+		(exclude_from_sim no)
+		(in_bom yes)
+		(on_board yes)
+		(dnp no)
+		(fields_autoplaced yes)
+		(property "Reference" "#PWR014"
+			(at 247.65 72.39 0)
+			(effects
+				(font
+					(size 1.27 1.27)
+				)
+				(hide yes)
+			)
+		)
+		(property "Value" "+5V_JETSON"
+			(at 247.65 63.5 0)
+			(effects
+				(font
+					(size 1.27 1.27)
+				)
+			)
+		)
+		(property "Footprint" ""
+			(at 247.65 68.58 0)
+			(effects
+				(font
+					(size 1.27 1.27)
+				)
+				(hide yes)
+			)
+		)
+		(property "Datasheet" ""
+			(at 247.65 68.58 0)
+			(effects
+				(font
+					(size 1.27 1.27)
+				)
+				(hide yes)
+			)
+		)
+		(property "Description" "Power symbol creates a global label with name \"+5V_JETSON\""
+			(at 247.65 68.58 0)
+			(effects
+				(font
+					(size 1.27 1.27)
+				)
+				(hide yes)
+			)
+		)
+		(pin "1"
+		)
+		(instances
+			(project "gamma_carrier"
+				(path "/14709545-fb6c-4e0b-b295-f7f5e8a286ba/0e58818c-005b-4d62-adc6-0567728bdecf"
+					(reference "#PWR014")
+					(unit 1)
+				)
+			)
+		)
+	)
+	(symbol
 		(lib_id "power:PWR_FLAG")
 		(at 135.89 57.15 0)
@@
 					(unit 1)
 				)
-			)
-		)
-	)
-	(symbol
-		(lib_id "power:+5V")
-		(at 224.79 68.58 0)
-		(unit 1)
-		(exclude_from_sim no)
-		(in_bom yes)
-		(on_board yes)
-		(dnp no)
-		(fields_autoplaced yes)
-		(property "Reference" "#PWR08"
-			(at 224.79 72.39 0)
-			(effects
-				(font
-					(size 1.27 1.27)
-				)
-				(hide yes)
-			)
-		)
-		(property "Value" "+5V"
-			(at 224.79 63.5 0)
-			(effects
-				(font
-					(size 1.27 1.27)
-				)
-			)
-		)
-		(property "Footprint" ""
-			(at 224.79 68.58 0)
-			(effects
-				(font
-					(size 1.27 1.27)
-				)
-				(hide yes)
-			)
-		)
-		(property "Datasheet" ""
-			(at 224.79 68.58 0)
-			(effects
-				(font
-					(size 1.27 1.27)
-				)
-				(hide yes)
-			)
-		)
-		(property "Description" "Power symbol creates a global label with name \"+5V\""
-			(at 224.79 68.58 0)
-			(effects
-				(font
-					(size 1.27 1.27)
-				)
-				(hide yes)
-			)
-		)
-		(pin "1"
-		)
-		(instances
-			(project ""
-				(path "/14709545-fb6c-4e0b-b295-f7f5e8a286ba/0e58818c-005b-4d62-adc6-0567728bdecf"
-					(reference "#PWR08")
-					(unit 1)
-				)
